File: pcb/masthead/masthead.kicad_pcb (KiCad board)
At the start: 2 copper layers, 48.6 x 56.5 mm, 10 parts, among them J1 Screw_Terminal_01x01, J2 Screw_Terminal_01x01, SW1 TILT, U1 TSR_1-2450, U2 WeMos_mini

Commit message: Tweaks
Parts:
- added U3: BMP580, PDJR_Module:BMP581, F.Cu at (15.4, 15.5)
Routing:
- net Net-(R2-Pad2): track 47.5 -> 74.2 mm, vias 0 -> 2
- net Net-(R3-Pad2): track 43.5 -> 70.0 mm
- net +3V3: track 0.00 -> 5.11 mm
- net GND: track 0.00 -> 4.94 mm, vias 0 -> 1
Changed lines of the file:
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@@
     (thickness 1.6)
     (drawings 143)
-    (tracks 39)
+    (tracks 65)
     (zones 0)
-    (modules 10)
-    (nets 18)
+    (modules 11)
+    (nets 20)
   )
   (page A4)
@@
   (net 16 "Net-(U2-Pad4)")
   (net 17 +5V)
+  (net 18 "Net-(U3-Pad5)")
+  (net 19 "Net-(U3-Pad3)")
   (net_class Default "This is the default net class."
     (clearance 0.2)
@@
     (add_net "Net-(U2-Pad8)")
     (add_net "Net-(U2-Pad9)")
+    (add_net "Net-(U3-Pad3)")
+    (add_net "Net-(U3-Pad5)")
   )
   (net_class Mains ""
@@
     (uvia_dia 0.3)
     (uvia_drill 0.1)
+  )
+  (module PDJR_Module:BMP581 (layer F.Cu)
+    (at 15.4 15.5)
+    (fp_text reference U3 (at 0 -1.95) (layer F.SilkS)
+      (effects (font (size 1 1) (thickness 0.15)))
+    )
+    (fp_text value BMP580 (at 0 2.05) (layer F.Fab)
+      (effects (font (size 1 1) (thickness 0.15)))
+    )
+    (fp_line (start -1 -1) (end 1 -1) (layer F.CrtYd) (width 0.12))
+    (fp_line (start 1 -1) (end 1 1) (layer F.CrtYd) (width 0.12))
+    (fp_line (start -1 -1) (end -1 1) (layer F.CrtYd) (width 0.12))
+    (fp_line (start -1 1) (end 1 1) (layer F.CrtYd) (width 0.12))
+    (fp_line (start -1.15 -1.15) (end 1.15 -1.15) (layer F.SilkS) (width 0.12))
+    (fp_line (start -1.15 -1.15) (end -1.15 1.15) (layer F.SilkS) (width 0.12))
+    (fp_line (start -1.15 1.15) (end 1.15 1.15) (layer F.SilkS) (width 0.12))
+    (fp_line (start 1.15 1.15) (end 1.15 -1.15) (layer F.SilkS) (width 0.12))
+    (pad 6 smd rect (at 0.765 0.25) (size 0.275 0.25) (layers F.Cu F.Paste F.Mask)
+      (net 2 +3V3))
+    (pad 7 smd rect (at 0.765 -0.25) (size 0.275 0.25) (layers F.Cu F.Paste F.Mask)
+      (net 1 GND))
+    (pad 2 smd rect (at -0.765 0.25) (size 0.275 0.25) (layers F.Cu F.Paste F.Mask)
+      (net 6 "Net-(R3-Pad2)"))
+    (pad 1 smd rect (at -0.765 -0.25) (size 0.275 0.25) (layers F.Cu F.Paste F.Mask)
+      (net 2 +3V3))
+    (pad 5 smd rect (at 0.5 0.7625) (size 0.25 0.275) (layers F.Cu F.Paste F.Mask)
+      (net 18 "Net-(U3-Pad5)"))
+    (pad 3 smd rect (at -0.5 0.7625) (size 0.25 0.275) (layers F.Cu F.Paste F.Mask)
+      (net 19 "Net-(U3-Pad3)"))
+    (pad 4 smd rect (at 0 0.7625) (size 0.25 0.275) (layers F.Cu F.Paste F.Mask)
+      (net 5 "Net-(R2-Pad2)"))
+    (pad 8 smd rect (at 0.5 -0.7625) (size 0.25 0.275) (layers F.Cu F.Paste F.Mask)
+      (net 1 GND))
+    (pad 10 smd rect (at -0.5 -0.7625) (size 0.25 0.275) (layers F.Cu F.Paste F.Mask)
+      (net 2 +3V3))
+    (pad 9 smd rect (at 0 -0.7625) (size 0.25 0.275) (layers F.Cu F.Paste F.Mask)
+      (net 1 GND))
   )
   (module Connector_PinSocket_2.54mm:PinSocket_1x02_P2.54mm_Vertical (layer F.Cu)
@@
     (effects (font (size 3.5 3.5) (thickness 0.875)))
   )
-  (segment (start 11.3 11.9) (end 11.5 11.7) (width 1) (layer B.Cu) (net 17))
-  (segment (start -10.52 11.9) (end 11.3 11.9) (width 1) (layer B.Cu) (net 17))
-  (segment (start -10.52 22.47) (end -11.43 23.38) (width 1) (layer B.Cu) (net 17))
-  (segment (start -10.52 11.9) (end -10.52 22.47) (width 1) (layer B.Cu) (net 17))
+  (via (at 17 14) (size 0.8) (drill 0.4) (layers F.Cu B.Cu) (net 1))
+  (segment (start 16.165 15.25) (end 16.75 15.25) (width 0.25) (layer F.Cu) (net 1))
+  (segment (start 17 15) (end 17 14) (width 0.25) (layer F.Cu) (net 1))
+  (segment (start 16.75 15.25) (end 17 15) (width 0.25) (layer F.Cu) (net 1))
+  (segment (start 15.4 14.7375) (end 15.4 14.2) (width 0.25) (layer F.Cu) (net 1))
+  (segment (start 15.4 14.2) (end 15.6 14) (width 0.25) (layer F.Cu) (net 1))
+  (segment (start 15.9 14.1) (end 15.8 14) (width 0.25) (layer F.Cu) (net 1))
+  (segment (start 15.9 14.7375) (end 15.9 14.1) (width 0.25) (layer F.Cu) (net 1))
+  (segment (start 15.8 14) (end 17 14) (width 0.25) (layer F.Cu) (net 1))
+  (segment (start 15.6 14) (end 15.8 14) (width 0.25) (layer F.Cu) (net 1))
+  (segment (start 14.635 15.25) (end 13.05 15.25) (width 0.25) (layer F.Cu) (net 2))
+  (segment (start 16.165 15.75) (end 17.95 15.75) (width 0.25) (layer F.Cu) (net 2))
+  (segment (start 14.9 14.7375) (end 14.9 13) (width 0.25) (layer F.Cu) (net 2))
   (segment (start -15.6 5.6) (end -13.5 3.5) (width 1) (layer B.Cu) (net 3))
   (segment (start -15.6 11.9) (end -15.6 5.6) (width 1) (layer B.Cu) (net 3))
@@
   (segment (start -11.43 33.54) (end -11.43 33.57) (width 0.25) (layer F.Cu) (net 5))
   (segment (start -13.3 35.41) (end -11.43 33.54) (width 0.25) (layer F.Cu) (net 5))
+  (segment (start -13.3 42) (end -13.3 35.41) (width 0.25) (layer F.Cu) (net 5))
   (segment (start -12.3 43) (end -13.3 42) (width 0.25) (layer F.Cu) (net 5))
-  (segment (start -13.3 42) (end -13.3 35.41) (width 0.25) (layer F.Cu) (net 5))
-  (segment (start 19.375472 43) (end -12.3 43) (width 0.25) (layer F.Cu) (net 5))
-  (segment (start 19.902022 43.52655) (end 19.375472 43) (width 0.25) (layer F.Cu) (net 5))
+  (segment (start 14.3 43) (end -12.3 43) (width 0.25) (layer F.Cu) (net 5))
+  (segment (start 19.375472 43) (end 19.902022 43.52655) (width 0.25) (layer F.Cu) (net 5))
+  (segment (start 14.3 43) (end 19.375472 43) (width 0.25) (layer F.Cu) (net 5))
+  (segment (start 15.4 16.2625) (end 15.4 22.9) (width 0.25) (layer F.Cu) (net 5))
+  (segment (start 15.4 22.9) (end 15.4 32.9) (width 0.25) (layer F.Cu) (net 5))
+  (segment (start 15.4 32.9) (end 15.4 39.8) (width 0.25) (layer F.Cu) (net 5))
+  (segment (start 15.4 39.8) (end 15.4 39.8) (width 0.25) (layer F.Cu) (net 5))
+  (via (at 15.4 39.8) (size 0.8) (drill 0.4) (layers F.Cu B.Cu) (net 5))
+  (via (at 15.4 43) (size 0.8) (drill 0.4) (layers F.Cu B.Cu) (net 5))
+  (segment (start 15.4 39.8) (end 15.4 43) (width 0.25) (layer B.Cu) (net 5))
   (segment (start 24.506065 41.379649) (end 24.506065 41.306065) (width 0.25) (layer F.Cu) (net 6))
   (segment (start 24.506065 41.306065) (end 24.1 40.9) (width 0.25) (layer F.Cu) (net 6))
-  (segment (start 24.1 40.9) (end 14.8 40.9) (width 0.25) (layer F.Cu) (net 6))
   (segment (start 14.8 40.9) (end 13.2 42.5) (width 0.25) (layer F.Cu) (net 6))
   (segment (start -8.07 36.08) (end -8.05 36.1) (width 0.25) (layer F.Cu) (net 6))
@@
   (segment (start -2.2 42.5) (end -2.8 42.5) (width 0.25) (layer F.Cu) (net 6))
   (segment (start 13.2 42.5) (end -2.2 42.5) (width 0.25) (layer F.Cu) (net 6))
+  (segment (start 15.9 40.9) (end 14.8 40.9) (width 0.25) (layer F.Cu) (net 6))
+  (segment (start 24.1 40.9) (end 15.9 40.9) (width 0.25) (layer F.Cu) (net 6))
+  (segment (start 14 15.9) (end 14 29.7) (width 0.25) (layer F.Cu) (net 6))
+  (segment (start 14 29.7) (end 14 41.7) (width 0.25) (layer F.Cu) (net 6))
+  (segment (start 14.15 15.75) (end 14 15.9) (width 0.25) (layer F.Cu) (net 6))
+  (segment (start 14.635 15.75) (end 14.15 15.75) (width 0.25) (layer F.Cu) (net 6))
   (segment (start 11.43 31) (end 11.43 30.97) (width 0.25) (layer F.Cu) (net 15))
   (segment (start -11.43 31) (end -11.4 31) (width 0.25) (layer F.Cu) (net 16))
+  (segment (start 11.3 11.9) (end 11.5 11.7) (width 1) (layer B.Cu) (net 17))
+  (segment (start -10.52 11.9) (end 11.3 11.9) (width 1) (layer B.Cu) (net 17))
+  (segment (start -10.52 22.47) (end -11.43 23.38) (width 1) (layer B.Cu) (net 17))
+  (segment (start -10.52 11.9) (end -10.52 22.47) (width 1) (layer B.Cu) (net 17))
   (zone (net 3) (net_name "Net-(J1-Pad1)") (layer F.Cu) (hatch edge 0.508)
     (priority 2)
@@
       )
     )
+  )
+  (zone (net 0) (net_name "") (layer F.Mask) (hatch edge 0.508)
+    (connect_pads (clearance 0.508))
+    (min_thickness 0.254)
+    (fill yes (arc_segments 32) (thermal_gap 0.508) (thermal_bridge_width 0.508))
+    (polygon
+      (pts
+        (xy 16.6 16.7) (xy 14.2 16.7) (xy 14.2 14.3) (xy 16.6 14.3)
+      )
+    )
