File: pcb/masthead/masthead.sch (KiCad schematic (older format))
At the start: 10 parts, among them J1 Screw_Terminal_01x01, J2 Screw_Terminal_01x01, SW1 TILT, U1 TSR_1-2450, U2 WeMos_mini

Commit message: Tweaks
Parts:
- added U3: BMP580, PDJR_Module:BMP581, symbol PDJR_Module:BMP580
Connections:
- net +3V3: now also U3.1 (VDDIO), U3.10 (VDD), U3.6 (CSB)
- net GND: now also U3.3 (VSS), U3.7 (INT), U3.8 (VSS), U3.9 (VSS)
- net at R2.2, RH1.2 (SDA), U2.5 (D2): now also U3.4 (SDI)
- net at R3.2, RH1.4 (SCL), U2.6 (D1): now also U3.2 (SCK)
- no-connect marks 10 -> 11
Other:
- moved on the sheet: RH1
Changed lines of the file:
@@
 $EndDescr
 $Comp
-L power:GND #PWR01
+L power:GND #PWR03
 U 1 1 65AA0461
-P 7500 4700
-F 0 "#PWR01" H 7500 4450 50  0001 C CNN
-F 1 "GND" V 7500 4500 50  0000 C CNN
-F 2 "" H 7500 4700 50  0001 C CNN
-F 3 "" H 7500 4700 50  0001 C CNN
-	1    7500 4700
+P 10200 4700
+F 0 "#PWR03" H 10200 4450 50  0001 C CNN
+F 1 "GND" V 10200 4500 50  0000 C CNN
+F 2 "" H 10200 4700 50  0001 C CNN
+F 3 "" H 10200 4700 50  0001 C CNN
+	1    10200 4700
 	0    -1   -1   0
 $EndComp
@@
 L pdjr:AM2320 RH1
 U 1 1 65B8C1AB
-P 7900 3750
-F 0 "RH1" H 8160 3803 60  0000 L CNN
-F 1 "AM2320" H 8160 3697 60  0000 L CNN
-F 2 "Connector_PinSocket_2.54mm:PinSocket_1x04_P2.54mm_Vertical" V 7525 3775 60  0001 C CNN
-F 3 "" V 7525 3775 60  0000 C CNN
-	1    7900 3750
-	1    0    0    -1
+P 8300 2950
+F 0 "RH1" V 8700 2950 60  0000 C CNN
+F 1 "AM2320" V 8600 2950 60  0000 C CNN
+F 2 "Connector_PinSocket_2.54mm:PinSocket_1x04_P2.54mm_Vertical" V 7925 2975 60  0001 C CNN
+F 3 "" V 7925 2975 60  0000 C CNN
+	1    8300 2950
+	0    -1   -1   0
 $EndComp
 NoConn ~ 6400 4000
 NoConn ~ 6400 4100
 Wire Wire Line
-	7100 3900 7500 3900
-Wire Wire Line
-	6800 3800 7500 3800
-Wire Wire Line
-	7400 3700 7500 3700
-Wire Wire Line
-	7400 3700 7400 4700
-Wire Wire Line
 	7100 2900 7400 2900
-Wire Wire Line
-	7500 3600 7400 3600
 Wire Wire Line
 	7400 3600 7400 2900
@@
 Wire Wire Line
 	5300 2900 5300 3400
-Wire Wire Line
-	7500 4700 7400 4700
-Connection ~ 7400 4700
 Connection ~ 6500 4700
 NoConn ~ 5400 3700
@@
 	6400 3900 7100 3900
 Wire Wire Line
-	6500 4700 7400 4700
-Wire Wire Line
 	5300 2900 6800 2900
 Wire Wire Line
 	5050 4700 6500 4700
 $Comp
-L power:+5V #PWR?
+L power:+5V #PWR01
 U 1 1 65B82C7A
 P 7500 2750
-F 0 "#PWR?" H 7500 2600 50  0001 C CNN
+F 0 "#PWR01" H 7500 2600 50  0001 C CNN
 F 1 "+5V" V 7515 2878 50  0000 L CNN
 F 2 "" H 7500 2750 50  0001 C CNN
@@
 	6500 2750 7500 2750
 Connection ~ 6500 2750
+Wire Wire Line
+	8150 3600 8150 3350
+Wire Wire Line
+	7400 3600 8150 3600
+Wire Wire Line
+	8350 3800 8350 3350
+Wire Wire Line
+	6800 3800 8350 3800
+Wire Wire Line
+	8450 3900 8450 3350
+Wire Wire Line
+	7100 3900 8450 3900
+Wire Wire Line
+	6500 4700 8250 4700
+Wire Wire Line
+	8250 3350 8250 4700
+Connection ~ 8250 4700
+Connection ~ 8350 3800
+Connection ~ 8450 3900
+Connection ~ 8150 3600
+$Comp
+L PDJR_Module:BMP580 U3
+U 1 1 65BA4BA8
+P 9500 2950
+F 0 "U3" H 9500 3450 50  0000 C CNN
+F 1 "BMP580" H 9500 3350 50  0000 C CNN
+F 2 "PDJR_Module:BMP581" H 9150 3200 50  0001 C CNN
+F 3 "" H 9150 3200 50  0001 C CNN
+	1    9500 2950
+	1    0    0    -1
+$EndComp
+Wire Wire Line
+	8250 4700 9050 4700
+Wire Wire Line
+	9550 3900 9550 3300
+Wire Wire Line
+	8450 3900 9550 3900
+Wire Wire Line
+	9650 3800 9650 3300
+Wire Wire Line
+	8350 3800 9650 3800
+Wire Wire Line
+	9350 3600 9350 3300
+Wire Wire Line
+	8150 3600 8950 3600
+Wire Wire Line
+	9450 3300 9450 4700
+Connection ~ 9450 4700
+Wire Wire Line
+	9450 4700 9950 4700
+Wire Wire Line
+	9150 2800 9050 2800
+Wire Wire Line
+	9050 2800 9050 2900
+Connection ~ 9050 4700
+Wire Wire Line
+	9050 4700 9450 4700
+Wire Wire Line
+	9150 2900 9050 2900
+Connection ~ 9050 2900
+Wire Wire Line
+	9050 2900 9050 4700
+Wire Wire Line
+	9150 2700 8950 2700
+Wire Wire Line
+	8950 2700 8950 3600
+Connection ~ 8950 3600
+Wire Wire Line
+	8950 3600 9350 3600
+Wire Wire Line
+	9850 2900 9950 2900
+Wire Wire Line
+	9950 2900 9950 4700
+Connection ~ 9950 4700
+Wire Wire Line
+	9950 4700 10200 4700
+NoConn ~ 9850 2700
+Wire Wire Line
+	8950 2700 8950 2300
+Wire Wire Line
+	8950 2300 9950 2300
+Wire Wire Line
+	9950 2300 9950 2800
+Wire Wire Line
+	9950 2800 9850 2800
+Connection ~ 8950 2700
 $EndSCHEMATC

Commit message: Tweaks
Parts:
- removed U3: BMP580, PDJR_Module:BMP581, symbol PDJR_Module:BMP580
- added U?: BMP580, symbol PDJR_Module:BMP580
Connections:
- net +3V3: now also U?.1 (VDDIO), U?.10 (VDD), U?.6 (CSB)
- net GND: now also U?.3 (VSS), U?.7 (INT), U?.8 (VSS), U?.9 (VSS)
- net at R2.2, RH1.2 (SDA), U2.5 (D2): now also U?.4 (SDI)
- net at R3.2, RH1.4 (SCL), U2.6 (D1): now also U?.2 (SCK)
Other:
- moved on the sheet: C1, J1, J2, R1, R2, R3, RH1, SW1, U1, U2

Commit message: Tweaks
Other:
- note removed: "Multisensor for monitoring temperature, pressure and mast state (up/down)."
Changed lines of the file:
@@
 Comment1 ""
 Comment2 ""
-Comment3 ""
-Comment4 ""
+Comment3 "Reports temperature, humidity, barometric pressure and mast state."
+Comment4 "https://github.com/pdjr-wemos/pdjr-mast-multisensor"
 $EndDescr
 $Comp
@@
 	4150 4250 4150 4600
 NoConn ~ 5500 4150
-Text Notes 7000 6650 0    50   ~ 0
-Multisensor for monitoring temperature, pressure and mast state (up/down).
 Wire Wire Line
 	5500 4250 5900 4250

Commit message: Finalise
Parts:
- removed U?: BMP580, symbol PDJR_Module:BMP580
- added U3: BMP581, PDJR_Module:BMP581, symbol PDJR_Module:BMP581
Connections:
- net +3V3: now also U3.1 (VDDIO), U3.10 (VDD), U3.6 (CSB)
- net GND: now also U3.3 (VSS), U3.7 (INT), U3.8 (VSS), U3.9 (VSS)
- net at R2.2, RH1.2 (SDA), U2.5 (D2): now also U3.4 (SDI)
- net at R3.2, RH1.4 (SCL), U2.6 (D1): now also U3.2 (SCK)
Changed lines of the file:
@@
 Connection ~ 8050 3150
 $Comp
-L PDJR_Module:BMP580 U?
-U 1 1 65BAD4A3
+L PDJR_Module:BMP581 U3
+U 1 1 65BBD5AE
 P 8600 3400
-F 0 "U?" H 8600 3915 50  0000 C CNN
-F 1 "BMP580" H 8600 3824 50  0000 C CNN
-F 2 "" H 8250 3650 50  0001 C CNN
+F 0 "U3" H 8600 3915 50  0000 C CNN
+F 1 "BMP581" H 8600 3824 50  0000 C CNN
+F 2 "PDJR_Module:BMP581" H 8250 3650 50  0001 C CNN
 F 3 "" H 8250 3650 50  0001 C CNN
 	1    8600 3400

Commit message: PCB tweak
Changed lines of the file:
@@
 Comp "PDJR"
 Comment1 ""
-Comment2 ""
+Comment2 "6.5 to 36 VDC input."
 Comment3 "Reports temperature, humidity, barometric pressure and mast state."
 Comment4 "https://github.com/pdjr-wemos/pdjr-mast-multisensor"
@@
 $EndComp
 $Comp
-L power:PWR_FLAG #FLG02
-U 1 1 65ACE77F
-P 2400 3600
-F 0 "#FLG02" H 2400 3675 50  0001 C CNN
-F 1 "PWR_FLAG" V 2400 3727 50  0001 L CNN
-F 2 "" H 2400 3600 50  0001 C CNN
-F 3 "~" H 2400 3600 50  0001 C CNN
-	1    2400 3600
-	-1   0    0    1
-$EndComp
-Wire Wire Line
-	2300 3600 2400 3600
-$Comp
 L power:+3V3 #PWR02
 U 1 1 65B3555F
@@
 	0    1    1    0
 $EndComp
-Connection ~ 2400 3600
 Wire Wire Line
 	2300 3200 2400 3200
@@
 $EndComp
 Wire Wire Line
-	2400 3600 3000 3600
-Wire Wire Line
 	3700 3600 3700 5150
 Connection ~ 3500 3200
@@
 	1    0    0    -1
 $EndComp
+Wire Wire Line
+	2300 3600 3000 3600
 $EndSCHEMATC

Commit message: Add VEML7700
Parts:
- added J3: VEML7700, Connector_JST:JST_SH_SM04B-SRSS-TB_1x04-1MP_P1.00mm_Horizontal, symbol Connector_Generic:Conn_01x04
Connections:
- net +3V3: now also J3.1 (Pin_1)
- net GND: now also J3.2 (Pin_2)
- net at R2.2, RH1.2 (SDA), U2.5 (D2)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: now also J3.3 (Pin_3)
- net at R3.2, RH1.4 (SCL), U2.6 (D1)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: now also J3.4 (Pin_4)
Changed lines of the file:
@@
 L power:GND #PWR03
 U 1 1 65AA0461
-P 9300 5150
-F 0 "#PWR03" H 9300 4900 50  0001 C CNN
-F 1 "GND" V 9300 4950 50  0000 C CNN
-F 2 "" H 9300 5150 50  0001 C CNN
-F 3 "" H 9300 5150 50  0001 C CNN
-	1    9300 5150
+P 10700 5150
+F 0 "#PWR03" H 10700 4900 50  0001 C CNN
+F 1 "GND" V 10700 4950 50  0000 C CNN
+F 2 "" H 10700 5150 50  0001 C CNN
+F 3 "" H 10700 5150 50  0001 C CNN
+	1    10700 5150
 	0    -1   -1   0
 $EndComp
@@
 Connection ~ 9050 5150
 Wire Wire Line
-	9050 5150 9300 5150
+	9050 5150 9700 5150
 NoConn ~ 8950 3150
 Wire Wire Line
@@
 Wire Wire Line
 	2300 3600 3000 3600
+$Comp
+L Connector_Generic:Conn_01x04 J3
+U 1 1 65BFF10F
+P 9700 3600
+F 0 "J3" V 9900 3600 50  0000 R CNN
+F 1 "VEML7700" V 9800 3750 50  0000 R CNN
+F 2 "Connector_JST:JST_SH_SM04B-SRSS-TB_1x04-1MP_P1.00mm_Horizontal" H 9700 3600 50  0001 C CNN
+F 3 "~" H 9700 3600 50  0001 C CNN
+	1    9700 3600
+	0    -1   -1   0
+$EndComp
+Wire Wire Line
+	8450 4050 9600 4050
+Wire Wire Line
+	9600 4050 9600 3800
+Connection ~ 8450 4050
+Wire Wire Line
+	9700 3800 9700 5150
+Connection ~ 9700 5150
+Wire Wire Line
+	9700 5150 10700 5150
+Wire Wire Line
+	8750 4250 9800 4250
+Wire Wire Line
+	9800 4250 9800 3800
+Connection ~ 8750 4250
+Wire Wire Line
+	8650 4350 9900 4350
+Wire Wire Line
+	9900 4350 9900 3800
+Connection ~ 8650 4350
 $EndSCHEMATC
