File: pcb/masthead/masthead.sch (KiCad schematic (older format))
At the start: 12 parts, among them J1 Screw_Terminal_01x01, J2 Screw_Terminal_01x01, J3 VEML7700, SW1 TILT, U1 TSR_1-2450, U2 WeMos_mini, U3 BMP581

Commit message: Tweaks
Parts:
- J1, J2: value Screw_Terminal_01x01 -> Open screw terminal 5x7
- J3: footprint Connector_JST:JST_SH_SM04B-SRSS-TB_1x04-1MP_P1.00mm_Horizontal -> PDJR_Module:VEML7700_SIDE
- RH1: footprint Connector_PinSocket_2.54mm:PinSocket_1x04_P2.54mm_Vertical -> PDJR_Sensor:AM2320_HORIZ
Connections:
- net +3V3: now also J3.2 (Pin_2); no longer J3.1 (Pin_1)
- net GND: now also J3.3 (Pin_3); no longer J3.2 (Pin_2)
- net SDA: now reaches R2.2, RH1.2 (SDA), U2.5 (D2), U3.4 (SDI)
- net SDA: now also J3.4 (Pin_4); no longer J3.3 (Pin_3)
- net SCL: now reaches R3.2, RH1.4 (SCL), U2.6 (D1), U3.2 (SCK)
- net SCL: now also J3.1 (Pin_1); no longer J3.4 (Pin_4)
Changed lines of the file:
@@
 F 0 "RH1" V 7250 3000 60  0000 C CNN
 F 1 "AM2320" V 7150 3000 60  0000 C CNN
-F 2 "Connector_PinSocket_2.54mm:PinSocket_1x04_P2.54mm_Vertical" V 6475 3025 60  0001 C CNN
+F 2 "PDJR_Sensor:AM2320_HORIZ" V 6475 3025 60  0001 C CNN
 F 3 "" V 6475 3025 60  0000 C CNN
 	1    6850 3000
@@
 P 1550 2800
 F 0 "J1" H 1550 2700 50  0000 C CNN
-F 1 "Screw_Terminal_01x01" H 1468 2666 50  0001 C CNN
+F 1 "Open screw terminal 5x7" H 1468 2666 50  0001 C CNN
 F 2 "PDJR_ScrewTerminal:M4_OPEN_TERMINAL" H 1550 2800 50  0001 C CNN
 F 3 "~" H 1550 2800 50  0001 C CNN
@@
 P 1550 3200
 F 0 "J2" H 1550 3100 50  0000 C CNN
-F 1 "Screw_Terminal_01x01" H 1468 3066 50  0001 C CNN
+F 1 "Open screw terminal 5x7" H 1468 3066 50  0001 C CNN
 F 2 "PDJR_ScrewTerminal:M4_OPEN_TERMINAL" H 1550 3200 50  0001 C CNN
 F 3 "~" H 1550 3200 50  0001 C CNN
@@
 	8500 2950 8500 4750
 Connection ~ 8500 4750
-Wire Wire Line
-	8500 4750 9150 4750
 NoConn ~ 8400 2750
 Wire Wire Line
@@
 F 0 "J3" V 9350 3200 50  0000 R CNN
 F 1 "VEML7700" V 9250 3350 50  0000 R CNN
-F 2 "Connector_JST:JST_SH_SM04B-SRSS-TB_1x04-1MP_P1.00mm_Horizontal" H 9150 3200 50  0001 C CNN
+F 2 "PDJR_Module:VEML7700_SIDE" H 9150 3200 50  0001 C CNN
 F 3 "~" H 9150 3200 50  0001 C CNN
 	1    9150 3200
@@
 $EndComp
 Wire Wire Line
-	7900 3650 9050 3650
-Wire Wire Line
-	9050 3650 9050 3400
+	7900 3650 9150 3650
 Connection ~ 7900 3650
-Wire Wire Line
-	9150 3400 9150 4750
-Connection ~ 9150 4750
-Wire Wire Line
-	9150 4750 10150 4750
-Wire Wire Line
-	8200 3850 9250 3850
-Wire Wire Line
-	9250 3850 9250 3400
 Connection ~ 8200 3850
 Wire Wire Line
-	8100 3950 9350 3950
-Wire Wire Line
-	9350 3950 9350 3400
+	8100 3950 9050 3950
 Connection ~ 8100 3950
+Wire Wire Line
+	8500 4750 9250 4750
+Text Label 5950 3950 0    50   ~ 0
+SCL
+Text Label 5950 3850 0    50   ~ 0
+SDA
+Wire Wire Line
+	9050 3400 9050 3950
+Wire Wire Line
+	9150 3400 9150 3650
+Wire Wire Line
+	9350 3850 9350 3400
+Wire Wire Line
+	8200 3850 9350 3850
+Wire Wire Line
+	9250 3400 9250 4750
+Connection ~ 9250 4750
+Wire Wire Line
+	9250 4750 10150 4750
 $EndSCHEMATC
